Commit message: refactor ur5 and wsg50
- add models/worlds to ur5_gazebo and install to gazebo path
- change structure of .xacro robots
- add 'parent' parameter to .xacro files
- add dynamic end-effectors to ur5.xacro
- <robot>.xacro are defined as macros, to be combined in e.g. ur5_gazebo
- add ur5.launch in ur5_gazebo
- matching order in .gazebo.xacro and .model.xacro
- create wsg50 package
- rename mesh files and links/joints
- add wsg50 JointEffortController
- add rotatum saturation
- add wsg50 controller interface
- add wsg50 config (ee_T_tcp)
- remove wsg dynamics
- tab indentation of .xacro files
- update meta-data of pkgs

File: ur5_description/robots/ur5.gazebo.xacro (robot description, xacro)
@@ -1,80 +1,86 @@
 <?xml version="1.0"?>
 <robot xmlns:xacro="http://www.ros.org/wiki/xacro">
-  <xacro:macro name="ur5_gazebo">
-    <!-- link 0 -->
-    <gazebo reference="ur5_link0">
-      <static>true</static>
-      <selfCollide>true</selfCollide>
-      <mu1>0.2</mu1>
-      <mu2>0.2</mu2>
-      <!-- <material>Gazebo/Grey</material> -->
-    </gazebo>
-    <!-- link/joint 1 -->
-    <gazebo reference="ur5_link1">
-	  <!-- <static>true</static> -->
-      <selfCollide>true</selfCollide>
-      <mu1>0.2</mu1>
-      <mu2>0.2</mu2>
-      <!-- <material>Gazebo/White</material> -->
-    </gazebo>
-    <gazebo reference="ur5_joint1">
-      <implicitSpringDamper>1</implicitSpringDamper>
-      <provideFeedback>true</provideFeedback>
-    </gazebo>
-    <!-- link/joint 2 -->
-    <gazebo reference="ur5_link2">
-      <selfCollide>true</selfCollide>
-      <mu1>0.2</mu1>
-      <mu2>0.2</mu2>
-      <!-- <material>Gazebo/White</material> -->
-    </gazebo>
-    <gazebo reference="ur5_joint2">
-      <implicitSpringDamper>1</implicitSpringDamper>
-      <provideFeedback>true</provideFeedback>
-    </gazebo>
-    <!-- link/joint 3 -->
-    <gazebo reference="ur5_link3">
-      <selfCollide>true</selfCollide>
-      <mu1>0.2</mu1>
-      <mu2>0.2</mu2>
-      <!-- <material>Gazebo/White</material> -->
-    </gazebo>
-    <gazebo reference="ur5_joint3">
-      <implicitSpringDamper>1</implicitSpringDamper>
-      <provideFeedback>true</provideFeedback>
-    </gazebo>
-    <!-- link/joint 4 -->
-    <gazebo reference="ur5_link4">
-      <selfCollide>true</selfCollide>
-      <mu1>0.2</mu1>
-      <mu2>0.2</mu2>
-      <!-- <material>Gazebo/White</material> -->
-    </gazebo>
-    <gazebo reference="ur5_joint4">
-      <implicitSpringDamper>1</implicitSpringDamper>
-      <provideFeedback>true</provideFeedback>
-    </gazebo>
-    <!-- link/joint 5 -->
-    <gazebo reference="ur5_link5">
-      <selfCollide>true</selfCollide>
-      <mu1>0.2</mu1>
-      <mu2>0.2</mu2>
-      <!-- <material>Gazebo/White</material> -->
-    </gazebo>
-    <gazebo reference="ur5_joint5">
-      <implicitSpringDamper>1</implicitSpringDamper>
-      <provideFeedback>true</provideFeedback>
-    </gazebo>
-    <!-- link/joint 6 -->
-    <gazebo reference="ur5_link6">
-      <selfCollide>true</selfCollide>
-      <mu1>0.2</mu1>
-      <mu2>0.2</mu2>
-      <!-- <material>Gazebo/White</material> -->
-    </gazebo>
-    <gazebo reference="ur5_joint6">
-      <implicitSpringDamper>1</implicitSpringDamper>
-      <provideFeedback>true</provideFeedback>
-    </gazebo>
-  </xacro:macro>
+<xacro:macro name="gazebo">
+	<!-- link 0 -->
+	<gazebo reference="link0">
+		<static>true</static>
+		<selfCollide>true</selfCollide>
+		<mu1>0.2</mu1>
+		<mu2>0.2</mu2>
+	</gazebo>
+	<!-- link/joint 1 -->
+	<gazebo reference="joint1">
+		<implicitSpringDamper>1</implicitSpringDamper>
+		<provideFeedback>true</provideFeedback>
+	</gazebo>
+	<gazebo reference="link1">
+	<!-- <static>true</static> -->
+		<selfCollide>true</selfCollide>
+		<mu1>0.2</mu1>
+		<mu2>0.2</mu2>
+	</gazebo>
+	<!-- link/joint 2 -->
+	<gazebo reference="joint2">
+		<implicitSpringDamper>1</implicitSpringDamper>
+		<provideFeedback>true</provideFeedback>
+	</gazebo>
+	<gazebo reference="link2">
+		<selfCollide>true</selfCollide>
+		<mu1>0.2</mu1>
+		<mu2>0.2</mu2>
+	</gazebo>
+	<!-- link/joint 3 -->
+	<gazebo reference="joint3">
+		<implicitSpringDamper>1</implicitSpringDamper>
+		<provideFeedback>true</provideFeedback>
+	</gazebo>
+	<gazebo reference="link3">
+		<selfCollide>true</selfCollide>
+		<mu1>0.2</mu1>
+		<mu2>0.2</mu2>
+	</gazebo>
+	<!-- link/joint 4 -->
+	<gazebo reference="joint4">
+		<implicitSpringDamper>1</implicitSpringDamper>
+		<provideFeedback>true</provideFeedback>
+	</gazebo>
+	<gazebo reference="link4">
+		<selfCollide>true</selfCollide>
+		<mu1>0.2</mu1>
+		<mu2>0.2</mu2>
+	</gazebo>
+	<!-- link/joint 5 -->
+	<gazebo reference="joint5">
+		<implicitSpringDamper>1</implicitSpringDamper>
+		<provideFeedback>true</provideFeedback>
+	</gazebo>
+	<gazebo reference="link5">
+		<selfCollide>true</selfCollide>
+		<mu1>0.2</mu1>
+		<mu2>0.2</mu2>
+	</gazebo>
+	<!-- link/joint 6 -->
+	<gazebo reference="joint6">
+		<implicitSpringDamper>1</implicitSpringDamper>
+		<provideFeedback>true</provideFeedback>
+	</gazebo>
+	<gazebo reference="link6">
+		<selfCollide>true</selfCollide>
+		<mu1>0.2</mu1>
+		<mu2>0.2</mu2>
+	</gazebo>
+	<!-- ee link/joint -->
+	<!-- <preserveFixedJoint> cancels joint reduction -->
+	<!-- https://github.com/osrf/gazebo/issues/2732 -->
+	<gazebo reference="joint_ee">
+		<implicitSpringDamper>1</implicitSpringDamper>
+		<provideFeedback>true</provideFeedback>
+		<preserveFixedJoint>true</preserveFixedJoint>
+	</gazebo>
+	 <gazebo reference="ee">
+		<selfCollide>true</selfCollide>
+		<mu1>0.2</mu1>
+		<mu2>0.2</mu2>
+	</gazebo>
+</xacro:macro>
 </robot>

File: ur5_description/robots/ur5.transmission.xacro (robot description, xacro)
@@ -1,86 +1,71 @@
 <?xml version="1.0"?>
 <robot xmlns:xacro="http://www.ros.org/wiki/xacro">
-  <xacro:macro name="ur5_transmission">
-    <!-- add planning scene -->
-    <gazebo>
-      <plugin filename="libgazebo_ros_moveit_planning_scene.so" name="gazebo_ros_moveit_planning_scene">
-        <topicName>/planning_scene</topicName>
-        <sceneName>workcell</sceneName>
-        <robotName>ur5</robotName>
-        <updatePeriod>0.5</updatePeriod>
-      </plugin>
-    </gazebo>
-    <!-- load Gazebo lib with desired parameters -->
-    <gazebo>
-      <plugin name="gazebo_ros_control" filename="libgazebo_ros_control.so">
-        <!-- <robotNamespace>/MYROBOT</robotNamespace> -->
-      </plugin>
-	  </gazebo>
-    <!-- transmission joint 1 -->
-    <transmission name="ur5_tran1">
-      <type>transmission_interface/SimpleTransmission</type>
-      <joint name="ur5_joint1">
-        <hardwareInterface>hardware_interface/EffortJointInterface</hardwareInterface>
-      </joint>
-      <actuator name="ur5_motor1">
-        <hardwareInterface>hardware_interface/EffortJointInterface</hardwareInterface>
-        <mechanicalReduction>1</mechanicalReduction>
-      </actuator>
-    </transmission>
-    <!-- transmission joint 2 -->
-    <transmission name="ur5_tran2">
-      <type>transmission_interface/SimpleTransmission</type>
-      <joint name="ur5_joint2">
-        <hardwareInterface>hardware_interface/EffortJointInterface</hardwareInterface>
-      </joint>
-      <actuator name="ur5_motor2">
-        <hardwareInterface>hardware_interface/EffortJointInterface</hardwareInterface>
-        <mechanicalReduction>1</mechanicalReduction>
-      </actuator>
-    </transmission>
-    <!-- transmission joint 3 -->
-    <transmission name="ur5_tran3">
-      <type>transmission_interface/SimpleTransmission</type>
-      <joint name="ur5_joint3">
-        <hardwareInterface>hardware_interface/EffortJointInterface</hardwareInterface>
-      </joint>
-      <actuator name="ur5_motor3">
-        <hardwareInterface>hardware_interface/EffortJointInterface</hardwareInterface>
-        <mechanicalReduction>1</mechanicalReduction>
-      </actuator>
-    </transmission>
-    <!-- transmission joint 4 -->
-    <transmission name="ur5_tran4">
-      <type>transmission_interface/SimpleTransmission</type>
-      <joint name="ur5_joint4">
-        <hardwareInterface>hardware_interface/EffortJointInterface</hardwareInterface>
-      </joint>
-      <actuator name="ur5_motor4">
-        <hardwareInterface>hardware_interface/EffortJointInterface</hardwareInterface>
-        <mechanicalReduction>1</mechanicalReduction>
-      </actuator>
-    </transmission>
-    <!-- transmission joint 5 -->
-    <transmission name="ur5_tran5">
-      <type>transmission_interface/SimpleTransmission</type>
-      <joint name="ur5_joint5">
-        <hardwareInterface>hardware_interface/EffortJointInterface</hardwareInterface>
-      </joint>
-      <actuator name="ur5_motor5">
-        <hardwareInterface>hardware_interface/EffortJointInterface</hardwareInterface>
-        <mechanicalReduction>1</mechanicalReduction>
-      </actuator>
-    </transmission>
-    <!-- transmission joint 6 -->
-    <transmission name="ur5_tran6">
-      <type>transmission_interface/SimpleTransmission</type>
-      <joint name="ur5_joint6">
-        <hardwareInterface>hardware_interface/EffortJointInterface</hardwareInterface>
-      </joint>
-      <actuator name="ur5_motor6">
-        <hardwareInterface>hardware_interface/EffortJointInterface</hardwareInterface>
-        <mechanicalReduction>1</mechanicalReduction>
-      </actuator>
-    </transmission>
-  </xacro:macro>
+<xacro:macro name="transmission" params="prefix:=''">
+	<!-- transmission joint 1 -->
+	<transmission name="tran1">
+		<type>transmission_interface/SimpleTransmission</type>
+		<joint name="joint1">
+			<hardwareInterface>hardware_interface/EffortJointInterface</hardwareInterface>
+		</joint>
+		<actuator name="motor1">
+			<hardwareInterface>hardware_interface/EffortJointInterface</hardwareInterface>
+			<mechanicalReduction>1</mechanicalReduction>
+		</actuator>
+	</transmission>
+	<!-- transmission joint 2 -->
+	<transmission name="tran2">
+		<type>transmission_interface/SimpleTransmission</type>
+		<joint name="joint2">
+			<hardwareInterface>hardware_interface/EffortJointInterface</hardwareInterface>
+		</joint>
+		<actuator name="motor2">
+			<hardwareInterface>hardware_interface/EffortJointInterface</hardwareInterface>
+			<mechanicalReduction>1</mechanicalReduction>
+		</actuator>
+	</transmission>
+	<!-- transmission joint 3 -->
+	<transmission name="tran3">
+		<type>transmission_interface/SimpleTransmission</type>
+		<joint name="joint3">
+			<hardwareInterface>hardware_interface/EffortJointInterface</hardwareInterface>
+		</joint>
+		<actuator name="motor3">
+			<hardwareInterface>hardware_interface/EffortJointInterface</hardwareInterface>
+			<mechanicalReduction>1</mechanicalReduction>
+		</actuator>
+	</transmission>
+	<!-- transmission joint 4 -->
+	<transmission name="tran4">
+		<type>transmission_interface/SimpleTransmission</type>
+		<joint name="joint4">
+			<hardwareInterface>hardware_interface/EffortJointInterface</hardwareInterface>
+		</joint>
+		<actuator name="motor4">
+			<hardwareInterface>hardware_interface/EffortJointInterface</hardwareInterface>
+			<mechanicalReduction>1</mechanicalReduction>
+		</actuator>
+	</transmission>
+	<!-- transmission joint 5 -->
+	<transmission name="tran5">
+		<type>transmission_interface/SimpleTransmission</type>
+		<joint name="joint5">
+			<hardwareInterface>hardware_interface/EffortJointInterface</hardwareInterface>
+		</joint>
+		<actuator name="motor5">
+			<hardwareInterface>hardware_interface/EffortJointInterface</hardwareInterface>
+			<mechanicalReduction>1</mechanicalReduction>
+		</actuator>
+	</transmission>
+	<!-- transmission joint 6 -->
+	<transmission name="tran6">
+		<type>transmission_interface/SimpleTransmission</type>
+		<joint name="joint6">
+			<hardwareInterface>hardware_interface/EffortJointInterface</hardwareInterface>
+		</joint>
+		<actuator name="motor6">
+			<hardwareInterface>hardware_interface/EffortJointInterface</hardwareInterface>
+			<mechanicalReduction>1</mechanicalReduction>
+		</actuator>
+	</transmission>
+</xacro:macro>
 </robot>
